File: VCU/Banc de test/Schematics_banc/Conversion_SPI_SDtoMCU.kicad_sch (KiCad schematic)
At the start: 17 parts, among them IC1 TPS73533DRVT, Q1 BSS138, Q24 BSS138, Q3 BSS138, Q4 BSS138

Commit message: Update schematic
Parts:
- removed C1: 10n, EPSA_lib:CAPC2012X130N, symbol EPSA_lib:Condensateur 0805Y1000104JXT
- removed C2: 22u, EPSA_lib:CAPC2012X130N, symbol EPSA_lib:Condensateur 0805Y1000104JXT
- removed C6: 4.7u, EPSA_lib:CAPC2012X130N, symbol EPSA_lib:Condensateur 0805Y1000104JXT
- removed IC1: TPS73533DRVT, SON65P200X200X80-7N, symbol Régulateur Linéaire 5V-3.3V:TPS73533DRVT
- added C4: 1u, EPSA_lib:CAPC2012X130N, symbol EPSA_lib:Condensateur 0805Y1000104JXT
- added IC1: TPS7B8633QDDARQ1, SOIC127P600X170-9N, symbol Régulateur de Tension Linéaire:TPS7B8633QDDARQ1
- added R62: 4k, EPSA_lib:RESC3216X70N, symbol EPSA_lib:Résistance RK73H2BLTDD2152F
- added R63: 1k, EPSA_lib:RESC3216X70N, symbol EPSA_lib:Résistance RK73H2BLTDD2152F
- C5: value 22u -> 2.2u
- renumbered Q3 to Q17, Q4 to Q18, Q24 to Q19, Q1 to Q20, R71 to R64, R72 to R65, R45 to R66, R13 to R67, R38 to R68, R39 to R69, R40 to R70, R12 to R71
Connections:
- net 3.3V: now also IC1.1 (OUT), R62.2
- net 5V: now also C4.2, IC1.7 (EN), IC1.8 (IN)
- net GND: now also C4.1, IC1.5 (GND_1), IC1.9 (GND_2), R63.2
- new net: IC1.2 (FB/NC), R62.1, R63.1
- no-connect marks 0 -> 3
Other:
- moved on the sheet: Q17, Q18, R64, R65, R68, R69

Commit message: Fin de stage
Parts:
- R62: value 4k -> 3k9
- R63: value 1k -> 910
- R64, R66, R67, R68, R70, R71: value 20k -> 18k
- R65, R69: value 10k -> 18k
Changed lines of the file:
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@@
 			)
 		)
-		(property "Value" "4k"
+		(property "Value" "3k9"
 			(at 128.27 38.0999 90)
 			(effects
@@
 		(property "Render Name" "Résistance"
 			(at 119.126 36.83 0)
+			(effects
+				(font
+					(size 1.27 1.27)
+				)
+				(hide yes)
+			)
+		)
+		(property "Sim.Type" ""
+			(at 125.73 45.72 0)
 			(effects
 				(font
@@
 			)
 		)
+		(property "Sim.Type" ""
+			(at 91.44 92.71 0)
+			(effects
+				(font
+					(size 1.27 1.27)
+				)
+				(hide yes)
+			)
+		)
 		(pin "2"
 		)
@@
 			)
 		)
-		(property "Value" "20k"
+		(property "Value" "18k"
 			(at 74.93 144.7799 90)
 			(effects
@@
 		(property "Render Name" "Résistance"
 			(at 65.786 143.51 0)
+			(effects
+				(font
+					(size 1.27 1.27)
+				)
+				(hide yes)
+			)
+		)
+		(property "Sim.Type" ""
+			(at 72.39 152.4 0)
 			(effects
 				(font
@@
 			)
 		)
-		(property "Value" "20k"
+		(property "Value" "18k"
 			(at 105.41 62.2299 90)
 			(effects
@@
 		(property "Render Name" "Résistance"
 			(at 96.266 60.96 0)
+			(effects
+				(font
+					(size 1.27 1.27)
+				)
+				(hide yes)
+			)
+		)
+		(property "Sim.Type" ""
+			(at 102.87 69.85 0)
 			(effects
 				(font
@@
 			)
 		)
+		(property "Sim.Type" ""
+			(at 91.44 62.23 0)
+			(effects
+				(font
+					(size 1.27 1.27)
+				)
+				(hide yes)
+			)
+		)
 		(pin "2"
 		)
@@
 			)
 		)
-		(property "Value" "20k"
+		(property "Value" "18k"
 			(at 80.01 62.2299 90)
 			(effects
@@
 		(property "Render Name" "Résistance"
 			(at 70.866 60.96 0)
+			(effects
+				(font
+					(size 1.27 1.27)
+				)
+				(hide yes)
+			)
+		)
+		(property "Sim.Type" ""
+			(at 77.47 69.85 0)
 			(effects
 				(font
@@
 			)
 		)
-		(property "Value" "10k"
+		(property "Value" "18k"
 			(at 80.01 92.7099 90)
 			(effects
@@
 		(property "Render Name" "Résistance"
 			(at 70.866 91.44 0)
+			(effects
+				(font
+					(size 1.27 1.27)
+				)
+				(hide yes)
+			)
+		)
+		(property "Sim.Type" ""
+			(at 77.47 100.33 0)
 			(effects
 				(font
@@
 			)
 		)
+		(property "Sim.Type" ""
+			(at 148.59 39.37 0)
+			(effects
+				(font
+					(size 1.27 1.27)
+				)
+				(hide yes)
+			)
+		)
 		(pin "1"
 		)
@@
 			)
 		)
+		(property "Sim.Type" ""
+			(at 87.63 118.11 0)
+			(effects
+				(font
+					(size 1.27 1.27)
+				)
+				(hide yes)
+			)
+		)
 		(pin "2"
 		)
@@
 			)
 		)
+		(property "Sim.Type" ""
+			(at 199.39 39.37 0)
+			(effects
+				(font
+					(size 1.27 1.27)
+				)
+				(hide yes)
+			)
+		)
 		(pin "1"
 		)
@@
 			)
 		)
-		(property "Value" "20k"
+		(property "Value" "18k"
 			(at 100.33 144.7799 90)
 			(effects
@@
 		(property "Render Name" "Résistance"
 			(at 91.186 143.51 0)
+			(effects
+				(font
+					(size 1.27 1.27)
+				)
+				(hide yes)
+			)
+		)
+		(property "Sim.Type" ""
+			(at 97.79 152.4 0)
 			(effects
 				(font
@@
 			)
 		)
+		(property "Sim.Type" ""
+			(at 86.36 144.78 0)
+			(effects
+				(font
+					(size 1.27 1.27)
+				)
+				(hide yes)
+			)
+		)
 		(pin "2"
 		)
@@
 			)
 		)
+		(property "Sim.Type" ""
+			(at 152.4 27.94 0)
+			(effects
+				(font
+					(size 1.27 1.27)
+				)
+				(hide yes)
+			)
+		)
 		(pin "1"
 		)
@@
 			)
 		)
-		(property "Value" "1k"
+		(property "Value" "910"
 			(at 138.43 41.91 0)
 			(effects
@@
 		(property "Render Name" "Résistance"
 			(at 138.43 39.116 0)
+			(effects
+				(font
+					(size 1.27 1.27)
+				)
+				(hide yes)
+			)
+		)
+		(property "Sim.Type" ""
+			(at 129.54 45.72 0)
 			(effects
 				(font
@@
 			)
 		)
-		(property "Value" "20k"
+		(property "Value" "18k"
 			(at 76.2 118.1099 90)
 			(effects
@@
 		(property "Render Name" "Résistance"
 			(at 67.056 116.84 0)
+			(effects
+				(font
+					(size 1.27 1.27)
+				)
+				(hide yes)
+			)
+		)
+		(property "Sim.Type" ""
+			(at 73.66 125.73 0)
 			(effects
 				(font
@@
 			)
 		)
-		(property "Value" "20k"
+		(property "Value" "18k"
 			(at 101.6 118.1099 90)
 			(effects
@@
 		(property "Render Name" "Résistance"
 			(at 92.456 116.84 0)
+			(effects
+				(font
+					(size 1.27 1.27)
+				)
+				(hide yes)
+			)
+		)
+		(property "Sim.Type" ""
+			(at 99.06 125.73 0)
 			(effects
 				(font
@@
 			)
 		)
-		(property "Value" "10k"
+		(property "Value" "18k"
 			(at 105.41 92.7099 90)
 			(effects
@@
 			(effects
 				(font
+					(size 1.27 1.27)
+				)
+				(hide yes)
+			)
+		)
+		(property "Sim.Type" ""
+			(at 102.87 100.33 0)
+			(effects
+				(font
