File: VCU/Banc de test/Schematics_banc/Schematics_banc.kicad_pcb (KiCad board)
At the start: 2 copper layers, 123 parts, among them IC1 TPS73533DRVT, J1 DM3AT-SF-PEJM5_40_, Q1 MMBF170, Q2 MMBF170, Q6 MMBF170, Q7 MMBF170, Q8 MMBF170, Q9 MMBF170

Commit message: Update schematic
Parts:
- removed 12V1: HSMC-C380, Footprints:HSMCC380
- removed AIR+1, AIR-1, BrakeLight1, BuzzerR2D1, Decharge1, Precharge1: LB_T64G-V2CA-59-Z484, Footprints:LBT64GV2CA59Z484
- removed AIR+_st1, AIR-_st1, R2D_Button1, TSON_Button5: 7914J-1-000E, Footprints:7914J1000E
- removed AIR+_st2, AIR-_st2, DryMode1, R2D_Button2, TSON_Button6: VFJD1105W-5C63A-TR, Footprints:LEDC3216X195N
- removed PS1: TEN_40-1211E, Footprints:TEN401211E
- removed PS2: TBA_1-0510, Footprints:TBA1
- removed the R10 at (194.4, 66.4)
- removed the R10 at (111.3, 117.0)
- removed the R12 at (200.1, 43.0)
- removed the R12 at (111.3, 120.3)
- removed the R13 at (200.1, 46.3)
- removed the R13 at (111.3, 123.7)
- removed the R14 at (200.1, 49.7)
- removed the R14 at (111.3, 127.0)
- removed the R16 at (117.0, 93.5)
- removed the R16 at (200.1, 56.4)
- removed the R18 at (117.0, 100.2)
- removed the R18 at (200.1, 59.7)
- removed the R2 at (194.4, 46.3)
- removed the R2 at (111.3, 93.5)
- removed the R22 at (117.0, 113.6)
- removed the R22 at (200.1, 63.1)
- removed the R23 at (200.1, 66.4)
- removed the R23 at (117.0, 117.0)
- removed the R24 at (200.1, 69.8)
- removed the R24 at (117.0, 120.3)
- removed the R25 at (205.8, 43.0)
- removed the R25 at (117.0, 123.7)
- removed the R26 at (117.0, 127.0)
- removed the R26 at (205.8, 46.3)
- removed the R27 at (122.8, 93.5)
- removed the R27 at (205.8, 49.7)
- removed the R28 at (205.8, 53.0)
- removed the R28 at (122.8, 96.8)
- removed the R29 at (205.8, 56.4)
- removed the R29 at (122.8, 100.2)
- removed the R38 at (194.4, 90.0)
- removed the R38 at (128.4, 93.5)
- removed the R39 at (128.4, 96.8)
- removed the R39 at (194.4, 93.4)
- removed the R40 at (194.4, 96.7)
- removed the R40 at (128.4, 100.2)
- removed the R41 at (205.8, 59.7)
- removed the R41 at (128.4, 103.5)
- removed the R42 at (205.8, 63.1)
- removed the R42 at (128.4, 106.9)
- removed the R43 at (205.8, 66.4)
- removed the R43 at (128.4, 110.2)
- removed the R44 at (205.8, 69.8)
- removed the R44 at (128.4, 113.6)
- removed the R5 at (111.3, 103.5)
- removed the R5 at (194.4, 49.7)
- removed the R6 at (194.4, 53.0)
- removed the R6 at (111.3, 106.9)
- removed the R8 at (111.3, 110.2)
- removed the R8 at (194.4, 59.7)
- removed the R9 at (111.3, 113.6)
- removed the R9 at (194.4, 63.1)
- added BLUE1: LB_T64G-V2CA-59-Z484, Footprints:LBT64GV2CA59Z484, F.Cu at (115.0, 94.0)
- added BLUE2: LB_T64G-V2CA-59-Z484, Footprints:LBT64GV2CA59Z484, F.Cu at (129.5, 94.0)
- added BLUE3: LB_T64G-V2CA-59-Z484, Footprints:LBT64GV2CA59Z484, F.Cu at (115.0, 99.0)
- added BLUE4: LB_T64G-V2CA-59-Z484, Footprints:LBT64GV2CA59Z484, F.Cu at (129.5, 99.0)
- added BLUE5: LB_T64G-V2CA-59-Z484, Footprints:LBT64GV2CA59Z484, F.Cu at (115.0, 104.0)
- added BLUE6: LB_T64G-V2CA-59-Z484, Footprints:LBT64GV2CA59Z484, F.Cu at (129.5, 104.0)
- added BLUE7: LB_T64G-V2CA-59-Z484, Footprints:LBT64GV2CA59Z484, F.Cu at (115.0, 109.0)
- added BLUE8: LB_T64G-V2CA-59-Z484, Footprints:LBT64GV2CA59Z484, F.Cu at (129.5, 109.0)
- added GREEN1: VFJD1105W-5C63A-TR, Footprints:LEDC3216X195N, F.Cu at (247.2, 41.9)
- added GREEN10: VFJD1105W-5C63A-TR, Footprints:LEDC3216X195N, F.Cu at (-2.00, 260.5)
- added GREEN11: VFJD1105W-5C63A-TR, Footprints:LEDC3216X195N, F.Cu at (-2.00, 264.2)
- added GREEN2: VFJD1105W-5C63A-TR, Footprints:LEDC3216X195N, F.Cu at (269.5, 41.5)
- added GREEN3: VFJD1105W-5C63A-TR, Footprints:LEDC3216X195N, F.Cu at (247.5, 53.0)
- added GREEN4: VFJD1105W-5C63A-TR, Footprints:LEDC3216X195N, F.Cu at (269.2, 52.0)
- added GREEN5: VFJD1105W-5C63A-TR, Footprints:LEDC3216X195N, F.Cu at (249.5, 65.0)
- added GREEN6: VFJD1105W-5C63A-TR, Footprints:LEDC3216X195N, F.Cu at (269.5, 65.5)
- added GREEN7: VFJD1105W-5C63A-TR, Footprints:LEDC3216X195N, F.Cu at (271.5, 77.0)
- added GREEN8: VFJD1105W-5C63A-TR, Footprints:LEDC3216X195N, F.Cu at (-2.00, 253.1)
- added GREEN9: VFJD1105W-5C63A-TR, Footprints:LEDC3216X195N, F.Cu at (-2.00, 256.8)
- added IC2: ATA6561-GBQW-N, Footprints:SON65P300X300X90-9N-D, F.Cu at (-9.74, 291.9)
- added IC3: TPS7B8633QDDARQ1, Footprints:SOIC127P600X170-9N, F.Cu at (36.7, 28.9)
- added J10: 4P Droit 22-11-2042, EPSA_lib:MOLEX_22-11-2042, F.Cu at (120.0, 193.5)
- added J11: DM3AT-SF-PEJM5_40_, Footprints:DM3ATSFPEJM540, F.Cu at (106.8, 180.4)
- added J2: 2P Droit 2-11-2022, EPSA_lib:MOLEX_22-11-2022, F.Cu at (255.5, 144.5)
- added J3: 4P Droit 22-11-2042, EPSA_lib:MOLEX_22-11-2042, F.Cu at (14.4, 262.5)
- added J4: 4P Droit 22-11-2042, EPSA_lib:MOLEX_22-11-2042, F.Cu at (14.4, 270.4)
- added J5: 6P Droit 22-11-2062, EPSA_lib:HDRV6W87P0X254_1X6_1509X635X1092P, F.Cu at (15.5, 134.2)
- added J6: 6P Droit 22-11-2062, EPSA_lib:HDRV6W87P0X254_1X6_1509X635X1092P, F.Cu at (15.5, 157.2)
- added J7: 10-97-7086, Footprints:HDRV8W87P254_2X4_1016X508X1055P, F.Cu at (121.0, 97.9)
- added J8: 10-97-7086, Footprints:HDRV8W87P254_2X4_1016X508X1055P, F.Cu at (279.7, 54.7)
- added J9: 2P Droit 2-11-2022, EPSA_lib:MOLEX_22-11-2022, F.Cu at (-5.09, 300.1)
- added Q10: SI2337DS-T1-BE3, EPSA_lib:SOT95P237X112-3N, F.Cu at (136.0, 86.0)
- added Q11: SI2337DS-T1-BE3, EPSA_lib:SOT95P237X112-3N, F.Cu at (105.0, 98.5)
- added Q12: SI2337DS-T1-BE3, EPSA_lib:SOT95P237X112-3N, F.Cu at (139.0, 95.5)
- added Q13: SI2337DS-T1-BE3, EPSA_lib:SOT95P237X112-3N, F.Cu at (105.0, 108.0)
- added Q14: SI2337DS-T1-BE3, EPSA_lib:SOT95P237X112-3N, F.Cu at (139.0, 104.5)
- added Q15: SI2337DS-T1-BE3, EPSA_lib:SOT95P237X112-3N, F.Cu at (114.5, 114.0)
- added Q16: SI2337DS-T1-BE3, EPSA_lib:SOT95P237X112-3N, F.Cu at (130.5, 115.5)
- added Q17: BSS138, Footprints:SOT95P240X120-3N, F.Cu at (125.7, 143.4)
- added Q18: BSS138, Footprints:SOT95P240X120-3N, F.Cu at (125.7, 148.1)
- added Q19: BSS138, Footprints:SOT95P240X120-3N, F.Cu at (125.7, 152.7)
- added Q20: BSS138, Footprints:SOT95P240X120-3N, F.Cu at (125.7, 157.4)
- added Q3: MMBF170, Footprints:SOT96P237X111-3N, B.Cu at (112.0, 98.5)
- added Q4: MMBF170, Footprints:SOT96P237X111-3N, B.Cu at (132.0, 98.5)
- added Q5: MMBF170, Footprints:SOT96P237X111-3N, B.Cu at (111.0, 103.5)
- added R10: 11k, EPSA_lib:RESC3216X70N, F.Cu at (35.0, 152.0)
- added R12: 11k, EPSA_lib:RESC3216X70N, F.Cu at (30.0, 175.0)
- added R13: 11k, EPSA_lib:RESC3216X70N, F.Cu at (35.1, 189.8)
- added R14: 600, EPSA_lib:RESC3216X70N, B.Cu at (120.0, 94.5)
- added R16: 600, EPSA_lib:RESC3216X70N, B.Cu at (116.5, 100.0)
- added R18: 600, EPSA_lib:RESC3216X70N, B.Cu at (116.0, 103.5)
- added R2: 21.5k, EPSA_lib:RESC3216X70N, F.Cu at (35.0, 114.5)
- added R22: 3k, EPSA_lib:RESC3216X70N, F.Cu at (118.0, 89.0)
- added R23: 3k, EPSA_lib:RESC3216X70N, F.Cu at (131.0, 85.5)
- added R24: 3k, EPSA_lib:RESC3216X70N, F.Cu at (105.0, 95.5)
- added R25: 3k, EPSA_lib:RESC3216X70N, F.Cu at (139.0, 99.0)
- added R26: 3k, EPSA_lib:RESC3216X70N, F.Cu at (105.0, 104.5)
- added R27: 3k, EPSA_lib:RESC3216X70N, F.Cu at (139.0, 108.0)
- added R28: 3k, EPSA_lib:RESC3216X70N, F.Cu at (118.0, 114.0)
- added R29: 3k, EPSA_lib:RESC3216X70N, F.Cu at (127.0, 115.5)
- added R38: 21.5k, EPSA_lib:RESC3216X70N, F.Cu at (250.2, 41.9)
- added R39: 21.5k, EPSA_lib:RESC3216X70N, F.Cu at (272.5, 41.5)
- added R40: 21.5k, EPSA_lib:RESC3216X70N, F.Cu at (250.5, 53.0)
- added R41: 21.5k, EPSA_lib:RESC3216X70N, F.Cu at (272.2, 52.0)
- added R42: 21.5k, EPSA_lib:RESC3216X70N, F.Cu at (252.5, 65.0)
- added R43: 21.5k, EPSA_lib:RESC3216X70N, F.Cu at (272.5, 65.5)
- added R44: 21.5k, EPSA_lib:RESC3216X70N, F.Cu at (274.5, 77.0)
- added R5: 21.5k, EPSA_lib:RESC3216X70N, F.Cu at (35.0, 163.0)
- added R6: 21.5k, EPSA_lib:RESC3216X70N, F.Cu at (34.5, 177.0)
- added R62: 4k, EPSA_lib:RESC3216X70N, F.Cu at (120.4, 142.7)
- added R63: 1k, EPSA_lib:RESC3216X70N, F.Cu at (120.4, 146.1)
- added R64: 20k, EPSA_lib:RESC3216X70N, F.Cu at (120.4, 149.4)
- added R65: 10k, EPSA_lib:RESC3216X70N, F.Cu at (120.4, 152.8)
- added R66: 20k, EPSA_lib:RESC3216X70N, F.Cu at (120.4, 156.1)
- added R67: 20k, EPSA_lib:RESC3216X70N, F.Cu at (120.4, 159.5)
- added R68: 20k, EPSA_lib:RESC3216X70N, F.Cu at (120.4, 162.8)
- added R69: 10k, EPSA_lib:RESC3216X70N, F.Cu at (120.4, 166.2)
- added R70: 20k, EPSA_lib:RESC3216X70N, F.Cu at (94.0, 185.0)
- added R71: 20k, EPSA_lib:RESC3216X70N, F.Cu at (96.0, 151.0)
- added R72: 4.7k, EPSA_lib:RESC3216X70N, F.Cu at (91.0, 175.0)
- added R73: 3k, EPSA_lib:RESC3216X70N, F.Cu at (37.5, 34.5)
- added R74: 3k, EPSA_lib:RESC3216X70N, F.Cu at (37.5, 37.9)
- added R8: 11k, EPSA_lib:RESC3216X70N, F.Cu at (35.0, 119.5)
- added R9: 11k, EPSA_lib:RESC3216X70N, F.Cu at (35.0, 135.6)
- added RED1: HSMC-C380, Footprints:HSMCC380, F.Cu at (33.0, 20.5)
- added S10: 100SP1T1B4M2QE, Footprints:100SP1T1B4M2QE, F.Cu at (240.3, 65.0)
- added S11: 7914J-1-000E, Footprints:7914J1000E, F.Cu at (264.5, 65.5)
- added S12: 7914J-1-000E, Footprints:7914J1000E, F.Cu at (266.2, 76.7)
- added S13: 7914J-1-000E, Footprints:7914J1000E, F.Cu at (-22.3, 273.5)
- added S14: 7914J-1-000E, Footprints:7914J1000E, F.Cu at (-12.5, 271.6)
- added S15: 7914J-1-000E, Footprints:7914J1000E, F.Cu at (-4.36, 271.6)
- added S16: 7914J-1-000E, Footprints:7914J1000E, F.Cu at (3.78, 271.6)
- added S17: 100SP1T1B4M2QE, Footprints:100SP1T1B4M2QE, F.Cu at (-33.7, 244.4)
- added S18: 100SP1T1B4M2QE, Footprints:100SP1T1B4M2QE, F.Cu at (-33.7, 253.9)
- added S19: 100SP1T1B4M2QE, Footprints:100SP1T1B4M2QE, F.Cu at (-33.7, 263.9)
- added S2: 100SP1T1B4M2QE, Footprints:100SP1T1B4M2QE, F.Cu at (28.5, 132.2)
- added S20: 100SP1T1B4M2QE, Footprints:100SP1T1B4M2QE, F.Cu at (-33.7, 273.8)
- added S3: 100SP1T1B4M2QE, Footprints:100SP1T1B4M2QE, F.Cu at (28.5, 148.5)
- added S4: 100SP1T1B4M2QE, Footprints:100SP1T1B4M2QE, F.Cu at (28.5, 165.0)
- added S5: 100SP1T1B4M2QE, Footprints:100SP1T1B4M2QE, F.Cu at (28.6, 186.3)
- added S6: 7914J-1-000E, Footprints:7914J1000E, F.Cu at (242.0, 41.5)
- added S7: 7914J-1-000E, Footprints:7914J1000E, F.Cu at (264.5, 41.5)
- added S8: 7914J-1-000E, Footprints:7914J1000E, F.Cu at (242.5, 53.0)
- added S9: 7914J-1-000E, Footprints:7914J1000E, F.Cu at (264.5, 52.3)
- added VR5: PTV09A-4015U-A503, Footprints:PTV09A4015UA503, F.Cu at (38.7, 183.8)
- C1: value 0.1u -> 15p; footprint Footprints:CAPC1608X90N -> EPSA_lib:CAPC2012X130N
- C2: value 22u -> 100n; footprint Footprints:CAPC1608X90N -> EPSA_lib:CAPC2012X130N
- C3: value 10n -> 4.7u; footprint Footprints:CAPC1608X90N -> EPSA_lib:CAPC2012X130N
- C4: value 4.7u -> 1u; footprint Footprints:CAPC1608X90N -> EPSA_lib:CAPC2012X130N
- C5: value 10u -> 2.2u
- IC1: value TPS73533DRVT -> TPS7B8633QDDARQ1; footprint Footprints:SON65P200X200X80-7N -> Footprints:SOIC127P600X170-9N
- J1: value DM3AT-SF-PEJM5_40_ -> 2P Angle 171857-4002; footprint Footprints:DM3ATSFPEJM540 -> EPSA_lib:1718574002
- Q1, Q2, Q6, Q7, Q8: moved to B.Cu
- Q9: value MMBF170 -> SI2337DS-T1-BE3; footprint Footprints:SOT96P237X111-3N -> EPSA_lib:SOT95P237X112-3N
- R1, R4, R7: value 15k -> 21.5k
- R11: value 3k -> 11k
- R15: value 8k2 -> 600; moved to B.Cu
- R17, R21: value 15k -> 600; moved to B.Cu
- R19, R20: value 21.5k -> 600; moved to B.Cu
- R30, R32, R34, R36: value 15k -> 3k
- R31, R33, R35, R37: value 21.5k -> 3k
- R45, R46, R47, R50, R51: value 8k2 -> 11k
- R48: value 600 -> 11k
- R49: value 3k9 -> 11k
- R52: value 600 -> 21.5k
- R53: value 3k9 -> 21.5k
- R54, R55: value 8k2 -> 21.5k
- R56, R58: value 15k -> 11k
- R57, R59: value 21.5k -> 11k
- R60: value 15k -> 4.7k
- R61: value 21.5k -> 4.7k
- moved R60 314.8 mm to (-7.69, 282.4)
- moved R61 314.8 mm to (-7.69, 285.7)
- moved R56 314.4 mm to (-19.6, 256.2)
- moved R57 314.4 mm to (-19.6, 259.5)
- moved R58 314.4 mm to (-19.6, 262.9)
- moved R59 314.4 mm to (-19.6, 266.2)
- moved C2 276.8 mm to (1.31, 288.9)
- moved C3 276.1 mm to (1.13, 290.9)
- moved C1 275.9 mm to (1.31, 286.0)
- moved VR4 241.0 mm to (38.6, 162.5), turned to -90 degrees
- moved S1 222.9 mm to (28.5, 116.5), turned to -90 degrees
- moved VR3 218.8 mm to (38.6, 146.0), turned to -90 degrees
- moved R52 207.5 mm to (-19.7, 242.9)
- moved R53 207.5 mm to (-19.7, 246.2)
- moved R54 207.5 mm to (-19.7, 249.6)
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Connections:
- C1 pad 1: unconnected-(C1-Pad1) -> GND
- C1 pad 2: unconnected-(C1-Pad2) -> CAN1RX
- C2 pad 1: /Conversion 5V-3.3V/3.3V -> GND
- C2 pad 2: GND -> 5V
- C3 pad 1: Net-(IC1-NR) -> GND
- C3 pad 2: GND -> Net-(C3-Pad2)
- C4 pad 1: /Conversion 5V-3.3V/5V -> GND
- C4 pad 2: unconnected-(C4-Pad2) -> 5V
- C5 pad 1: unconnected-(C5-Pad1) -> GND
- C5 pad 2: unconnected-(C5-Pad2) -> /Conversion 5V-3.3V/3.3V
- IC1 pad 2: Net-(IC1-NR) -> Net-(IC1-FB/NC)
- IC1 pad 3: GND -> unconnected-(IC1-NC_1-Pad3)
- IC1 pad 4: /Conversion 5V-3.3V/5V -> unconnected-(IC1-NC_2-Pad4)
- IC1 pad 5: unconnected-(IC1-NC-Pad5) -> GND
- IC1 pad 6: /Conversion 5V-3.3V/5V -> unconnected-(IC1-NC_3-Pad6)
- IC1 pad 7: unconnected-(IC1-EP-Pad7) -> 5V
- J1 pad 1: unconnected-(J1-DAT2-Pad1) -> 12V
- J1 pad 2: 3.3V -> GND
- Q1 pad 2: Net-(Decharge1-A) -> GND
- Q1 pad 3: 12V -> Net-(Q1-D)
- Q2 pad 2: Net-(Precharge1-A) -> GND
- Q2 pad 3: 12V -> Net-(Q10-G)
- Q6 pad 1: BuzzerR2D_cmd -> Net-(Q6-G)
- Q6 pad 2: Net-(BuzzerR2D1-A) -> GND
- Q6 pad 3: 12V -> Net-(Q14-G)
- Q7 pad 1: BrakeLight_cmd -> Net-(Q7-G)
- Q7 pad 2: Net-(BrakeLight1-A) -> GND
- Q7 pad 3: 12V -> Net-(Q15-G)
- Q8 pad 2: Net-(AIR+1-A) -> GND
- Q8 pad 3: 12V -> Net-(Q16-G)
- Q9 pad 1: Net-(Q9-G) -> Net-(Q1-D)
- Q9 pad 2: Net-(AIR-1-A) -> 12V
- Q9 pad 3: 12V -> Net-(Q9-D)
- R1 pad 1: APPS2 -> GND
- R1 pad 2: GND -> Net-(RED1-K)
- R15 pad 1: Decharge_cmd -> AIR-_cmd
- R15 pad 2: Net-(Q1-G) -> Net-(Q2-G)
- R17 pad 1: LV_BATT -> BuzzerR2D_cmd
- R17 pad 2: GND -> Net-(Q4-G)
- R19 pad 1: AIR+_st -> Decharge_cmd
- R19 pad 2: Net-(AIR+_st1-+_1) -> Net-(Q6-G)
- R20 pad 1: LV_BATT -> GPIO1
- R20 pad 2: 12V -> Net-(Q7-G)
- R21 pad 1: GND -> GPIO3
- R21 pad 2: AIR+_st -> Net-(Q8-G)
- R3 pad 1: APPS1 -> Net-(R3-Pad1)
- R3 pad 2: Net-(VR1-WIPER) -> Net-(VR2-WIPER)
- R30 pad 1: GND -> Net-(Q9-D)
- R30 pad 2: FRWSS -> Net-(BLUE1-A)
- R31 pad 1: FRWSS -> Net-(Q10-D)
- R32 pad 1: GND -> Net-(Q11-D)
- R32 pad 2: FLWSS -> Net-(BLUE3-A)
- R33 pad 1: FLWSS -> Net-(Q12-D)
- R34 pad 1: GND -> Net-(Q13-D)
- R34 pad 2: RLWSS -> Net-(BLUE5-A)
- R35 pad 1: RLWSS -> Net-(Q14-D)
- R36 pad 1: GND -> Net-(Q15-D)
- R36 pad 2: RRWSS -> Net-(BLUE7-A)
- R37 pad 1: RRWSS -> Net-(Q16-D)
- R4 pad 1: APPS1 -> Net-(R10-Pad1)
- R4 pad 2: GND -> Net-(VR3-WIPER)
- R45 pad 1: Net-(Q2-G) -> GND
- R45 pad 2: GND -> AIR+_st
- R46 pad 1: Net-(Q2-G) -> GND
- R46 pad 2: 5V -> AIR-_st
- R47 pad 1: Net-(Q3-G) -> GND
- R47 pad 2: GND -> TSON_Button
- R48 pad 1: Net-(AIR+1-K) -> GND
- R48 pad 2: Net-(Q4-D) -> R2D_Button
- R49 pad 1: AIR+_cmd -> GND
- R49 pad 2: Net-(Q4-G) -> Dry/WetSwitch_st
- R50 pad 1: Net-(Q4-G) -> GND
- R50 pad 2: 5V -> GPIO2
- R51 pad 1: Net-(Q4-G) -> GND
- R51 pad 2: GND -> GPIO4
- R52 pad 1: Net-(AIR-1-K) -> Net-(R52-Pad1)
- R53 pad 1: AIR-_cmd -> Net-(R53-Pad1)
- R53 pad 2: Net-(Q5-G) -> Net-(S14-+_1)
- R54 pad 1: Net-(Q5-G) -> Net-(R54-Pad1)
- R54 pad 2: 5V -> Net-(S15-+_1)
- R55 pad 1: Net-(Q5-G) -> Net-(R55-Pad1)
- R55 pad 2: GND -> Net-(S16-+_1)
- R56 pad 2: AIR-_st -> Net-(R52-Pad1)
- R57 pad 1: AIR-_st -> GND
- R57 pad 2: Net-(AIR-_st1-+_1) -> Net-(R53-Pad1)
- R58 pad 2: TSON_Button -> Net-(R54-Pad1)
- R59 pad 1: TSON_Button -> GND
- R59 pad 2: Net-(TSON_Button5-+_1) -> Net-(R55-Pad1)
- R60 pad 1: GND -> Net-(C3-Pad2)
- R60 pad 2: R2D_Button -> CAN1H
- R61 pad 1: R2D_Button -> CAN1L
- R61 pad 2: Net-(R2D_Button1-+_1) -> Net-(C3-Pad2)
- R7 pad 1: RBPS -> Net-(R13-Pad1)
- R7 pad 2: GND -> Net-(VR5-WIPER)
- S1 pad 1: 12V -> Net-(R2-Pad1)
- S1 pad 2: Net-(DryMode1-A) -> APPS1
- S1 pad 3: GND -> APPS1_EXT
Routing:
- net GND: track 0.00 -> 116.0 mm, vias 0 -> 8
- net 12V: track 0.00 -> 80.5 mm
- net APPS1_EXT: track 0.00 -> 47.5 mm
- net ADC5: track 0.00 -> 44.9 mm
- net LV_BATT: track 0.00 -> 41.4 mm
- net APPS2_EXT: track 0.00 -> 37.9 mm
- net AIR+_st: track 0.00 -> 37.1 mm
- net TSON_Button: track 0.00 -> 30.3 mm
- net Dry/WetSwitch_st: track 0.00 -> 29.8 mm
- net RBPS: track 0.00 -> 28.6 mm
- net ADC5_EXT: track 0.00 -> 26.5 mm
- net APPS1: track 0.00 -> 26.1 mm
- net FBPS: track 0.00 -> 19.7 mm
- net AIR-_st: track 0.00 -> 17.4 mm
- net GPIO4: track 0.00 -> 17.3 mm
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
Commit message: Routage Support de programmation VCU
Parts:
- added ?: , , F.Cu at (202.0, 29.5)
- added ?: , , F.Cu at (202.0, 141.0)
- added ?: , , F.Cu at (65.5, 29.5)
- added ?: , , F.Cu at (65.5, 140.5)
- added C6: 2.2u, EPSA_lib:CAPC2012X130N, F.Cu at (166.7, 40.7)
- added C7: 1u, EPSA_lib:CAPC2012X130N, F.Cu at (163.2, 40.7)
- added J12: DM3AT-SF-PEJM5_40_, Footprints:DM3ATSFPEJM540, B.Cu at (144.5, 54.0)
- C4, C5, IC1, Q17, Q18, Q19, Q20, R62, R63, R64, R65, R66, R67, R68, R69, R70, R71, R72: moved to B.Cu
- J10: value 4P Droit 22-11-2042 -> 2P Droit 2-11-2022; footprint EPSA_lib:MOLEX_22-11-2042 -> EPSA_lib:MOLEX_22-11-2022
- J11: value DM3AT-SF-PEJM5_40_ -> 4P Droit 22-11-2042; footprint Footprints:DM3ATSFPEJM540 -> EPSA_lib:MOLEX_22-11-2042
- R73: value 3k -> 13.3k
- R74: value 3k -> 2k
- moved J9 290.2 mm to (102.4, 30.6)
- moved R61 281.0 mm to (120.4, 35.6), turned to 180 degrees
- moved IC2 279.3 mm to (105.9, 37.6)
- moved C3 277.5 mm to (116.9, 38.6), turned to 90 degrees
- moved R60 274.9 mm to (113.4, 35.6), turned to 180 degrees
- moved C2 269.6 mm to (106.4, 40.6)
- moved C1 266.5 mm to (100.4, 38.6)
- moved S17 242.1 mm to (164.3, 105.0)
- moved S18 235.9 mm to (149.3, 105.0)
- moved S13 232.4 mm to (157.3, 126.0), turned to -90 degrees
- moved S19 230.8 mm to (133.8, 105.0)
- moved R56 228.9 mm to (157.8, 111.5), turned to 180 degrees
- moved S20 226.8 mm to (117.8, 105.0)
- moved R57 222.0 mm to (145.8, 111.5), turned to 180 degrees
- moved R52 219.0 mm to (157.8, 114.5)
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Connections:
- J10 pad 1: SS_SDC_5V -> CAN1H
- J10 pad 2: MISO_5V -> CAN1L
- J11 pad 1: unconnected-(J11-DAT2-Pad1) -> SS_SDC_5V
- J11 pad 2: /Conversion 5V-3.3V/SS_3.3V -> MISO_5V
- J11 pad 3: /Conversion 5V-3.3V/MISO_3.3V -> SCK_5V
- J11 pad 4: /Conversion 5V-3.3V/3.3V -> MOSI_5V
- J9 pad 1: CAN1H -> CAN1RX
- J9 pad 2: CAN1L -> CAN1TX
- R52 pad 2: Net-(S13-+_1) -> Net-(GREEN8-K)
- R53 pad 2: Net-(S14-+_1) -> Net-(GREEN9-K)
- R54 pad 2: Net-(S15-+_1) -> Net-(GREEN10-K)
- R55 pad 2: Net-(S16-+_1) -> Net-(GREEN11-K)
- S13 pad 2: Net-(GREEN8-A) -> 12V
- S13 pad 3: Net-(S13-+_1) -> Net-(GREEN8-A)
- S13 pad 4: Net-(GREEN8-K) -> Net-(GREEN8-A)
- S14 pad 2: Net-(GREEN9-A) -> 12V
- S14 pad 3: Net-(S14-+_1) -> Net-(GREEN9-A)
- S14 pad 4: Net-(GREEN9-K) -> Net-(GREEN9-A)
- S15 pad 2: Net-(GREEN10-A) -> 12V
- S15 pad 3: Net-(S15-+_1) -> Net-(GREEN10-A)
- S15 pad 4: Net-(GREEN10-K) -> Net-(GREEN10-A)
- S16 pad 2: Net-(GREEN11-A) -> 12V
- S16 pad 3: Net-(S16-+_1) -> Net-(GREEN11-A)
- S16 pad 4: Net-(GREEN11-K) -> Net-(GREEN11-A)
Routing:
- net GND: track 116.0 -> 239.1 mm, vias 8 -> 14
- net 5V: track 0.00 -> 59.4 mm, vias 0 -> 8
- net FRWSS_in: track 0.00 -> 48.8 mm
- net RLWSS_out: track 0.00 -> 44.1 mm
- net FLWSS_in: track 0.00 -> 42.9 mm
- net FRWSS_out: track 0.00 -> 42.6 mm
- net RRWSS_in: track 0.00 -> 37.5 mm
- net RRWSS_out: track 0.00 -> 36.9 mm
- net FLWSS_out: track 0.00 -> 36.5 mm
- net RLWSS_in: track 0.00 -> 36.0 mm
- net /Conversion 5V-3.3V/SS_3.3V: track 0.00 -> 24.6 mm
- net CAN1L: track 0.00 -> 22.2 mm
- net /Conversion 5V-3.3V/MISO_3.3V: track 0.00 -> 19.7 mm
- net /Conversion 5V-3.3V/SCK_3.3V: track 0.00 -> 15.0 mm
- net SS_SDC_5V: track 0.00 -> 14.9 mm
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- added copper zone on B.Cu, net /Conversion 5V-3.3V/3.3V
- added copper zone on F.Cu, net 12V
- added copper zone on F.Cu, net 5V
- added copper zone on B.Cu, net GND
Other:
- board outline added: 152.5 x 127 mm
- board text added: "1"
- board text added: "12V"
- board text added: "2"
- board text added: "5V"
- board text added: "7"
- board text added: "8"
- board text added: "ADC0"
- board text added: "ADC1"
- board text added: "ADC2"
- board text added: "ADC3"
- board text added: "ADC5"
- board text added: "Alimentation Externe 12V"
- board text added: "Alimentation MCU 5V"
- board text added: "CAN1H"
- board text added: "CAN1L"
- board text added: "CAN1RX"
- board text added: "CAN1TX"
- board text added: "Connecteur Micro-SD"
- board text added: "Entrées Analogiques Ext"
- board text added: "Entrées Analogiques Manuelles"
- board text added: "Entrées Compteurs Externes"
- board text added: "Entrées Compteurs Manuels"
- board text added: "G1"
- board text added: "G2"
- board text added: "G3"
- board text added: "G4"
- board text added: "G5"
- board text added: "G6"
- board text added: "G7"
- board text added: "G8"
- board text added: "GND"
- board text added: "Gestion Carte Micro-SD"
- board text added: "MISO"
- board text added: "MOSI"
- board text added: "SCK"
- board text added: "SS"
- board text added: "Sorties Digitales"
- board text added: "TC1"
- board text added: "TC2"
- board text added: "TC3"
- board text added: "TC4"
- board text added: "VDDANA"

Commit message: Routage Final
Parts:
- removed ? (x4): , 
- removed S1, S10, S17, S18, S19, S2, S20, S3, S4, S5: 100SP1T1B4M2QE, Footprints:100SP1T1B4M2QE
- removed S11, S12, S13, S14, S15, S16, S6, S7, S8, S9: 7914J-1-000E, Footprints:7914J1000E
- removed VR1, VR2, VR3, VR4, VR5: PTV09A-4015U-A503, Footprints:PTV09A4015UA503
- added M2: MountingHole_3.2mm_M3_DIN965_Pad, MountingHole:MountingHole_3.2mm_M3_DIN965_Pad, F.Cu at (64.0, 135.0)
- added M2: MountingHole_3.2mm_M3_DIN965_Pad, MountingHole:MountingHole_3.2mm_M3_DIN965_Pad, F.Cu at (64.0, 47.0)
- added M2: MountingHole_3.2mm_M3_DIN965_Pad, MountingHole:MountingHole_3.2mm_M3_DIN965_Pad, F.Cu at (200.0, 135.0)
- added M2: MountingHole_3.2mm_M3_DIN965_Pad, MountingHole:MountingHole_3.2mm_M3_DIN965_Pad, F.Cu at (200.0, 47.0)
- added RV1: R_Potentiometer, Footprints:PTV09A4015UA503, F.Cu at (95.0, 49.0)
- added RV2: R_Potentiometer, Footprints:PTV09A4015UA503, F.Cu at (95.1, 65.0)
- added RV3: R_Potentiometer, Footprints:PTV09A4015UA503, F.Cu at (95.1, 81.5)
- added RV4: R_Potentiometer, Footprints:PTV09A4015UA503, F.Cu at (95.1, 98.0)
- added RV5: R_Potentiometer, Footprints:PTV09A4015UA503, F.Cu at (95.1, 119.5)
- added SW1: 100SP1T1B4M2QE, Footprints:100SP1T1B4M2QE, F.Cu at (85.0, 52.0)
- added SW10: 100SP1T1B4M2QE, Footprints:100SP1T1B4M2QE, F.Cu at (182.9, 71.9)
- added SW11: 7914J-1-000E, Footprints:7914J1000E, F.Cu at (183.4, 48.3)
- added SW12: 7914J-1-000E, Footprints:7914J1000E, F.Cu at (196.5, 69.1)
- added SW13: 7914J-1-000E, Footprints:7914J1000E, F.Cu at (183.0, 90.9)
- added SW14: 7914J-1-000E, Footprints:7914J1000E, F.Cu at (183.2, 102.3)
- added SW15: 7914J-1-000E, Footprints:7914J1000E, F.Cu at (183.2, 114.3)
- added SW16: 7914J-1-000E, Footprints:7914J1000E, F.Cu at (183.0, 125.1)
- added SW17: 100SP1T1B4M2QE, Footprints:100SP1T1B4M2QE, F.Cu at (162.0, 83.1)
- added SW18: 100SP1T1B4M2QE, Footprints:100SP1T1B4M2QE, F.Cu at (162.2, 98.3)
- added SW19: 100SP1T1B4M2QE, Footprints:100SP1T1B4M2QE, F.Cu at (162.2, 113.7)
- added SW2: 100SP1T1B4M2QE, Footprints:100SP1T1B4M2QE, F.Cu at (85.0, 68.0)
- added SW20: 100SP1T1B4M2QE, Footprints:100SP1T1B4M2QE, F.Cu at (162.2, 129.7)
- added SW3: 100SP1T1B4M2QE, Footprints:100SP1T1B4M2QE, F.Cu at (85.0, 84.0)
- added SW4: 100SP1T1B4M2QE, Footprints:100SP1T1B4M2QE, F.Cu at (85.0, 100.5)
- added SW5: 100SP1T1B4M2QE, Footprints:100SP1T1B4M2QE, F.Cu at (85.0, 121.5)
- added SW6: 7914J-1-000E, Footprints:7914J1000E, F.Cu at (158.7, 69.7)
- added SW7: 7914J-1-000E, Footprints:7914J1000E, F.Cu at (159.2, 48.3)
- added SW8: 7914J-1-000E, Footprints:7914J1000E, F.Cu at (170.5, 69.2)
- added SW9: 7914J-1-000E, Footprints:7914J1000E, F.Cu at (170.2, 48.3)
- R64, R65, R66, R67: moved to F.Cu
- moved J4 68.8 mm to (192.4, 119.4), turned to -90 degrees
- moved J3 59.8 mm to (192.3, 100.2), turned to -90 degrees
- moved GREEN11 53.7 mm to (176.2, 124.7), turned to 0 degrees
- moved R55 49.9 mm to (171.7, 124.7), turned to 90 degrees
- moved R59 47.7 mm to (168.7, 124.7), turned to -90 degrees
- moved GREEN10 42.7 mm to (176.2, 113.7), turned to 0 degrees
- moved J2 40.6 mm to (112.0, 27.7)
- moved R64 39.0 mm to (110.7, 33.3)
- moved Q20 38.9 mm to (91.3, 34.0), turned to 180 degrees
- moved R54 38.4 mm to (172.2, 113.7), turned to 90 degrees
- moved C3 38.2 mm to (79.0, 33.8), turned to -90 degrees
- moved R65 38.1 mm to (104.6, 33.3)
- moved R60 38.0 mm to (75.5, 32.8)
- moved J10 38.0 mm to (77.5, 27.8)
- moved J9 38.0 mm to (64.5, 27.8)
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Routing:
- net 12V: track 80.8 -> 0.77 mm
- net GND: track 239.1 -> 195.6 mm, vias 14 -> 20
- net FRWSS_in: track 48.8 -> 82.7 mm
- net 5V: track 59.4 -> 30.3 mm, vias 8 -> 2
- net GPIO4: track 18.9 -> 40.8 mm
- net CAN1RX: track 11.7 -> 27.7 mm, vias 0 -> 1
- net CAN1TX: track 6.14 -> 18.3 mm
- net /Conversion 5V-3.3V/3.3V: track 11.9 -> 0.00 mm, vias 4 -> 0
- net Dry/WetSwitch_st: track 41.0 -> 31.0 mm
- net Net-(GREEN3-A): track 7.87 -> 16.3 mm
- net MOSI_5V: track 12.4 -> 19.8 mm, vias 0 -> 1
- net CAN1L: track 22.2 -> 16.9 mm
- net FBPS: track 19.7 -> 24.8 mm
- net FRWSS_out: track 42.6 -> 37.8 mm
- net LV_BATT: track 41.4 -> 45.9 mm
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Other:
- board size 152.5 x 127 mm -> 144.2 x 116.7 mm
