File: VCU/Banc de test/Schematics_banc/Schematics_banc.kicad_sch (KiCad schematic)
At the start: 136 parts, among them IC2 ATA6561-GBQW-N, J1 DM3AT-SF-PEJM5_40_, Q15 MMBF170, Q16 SI2337DS-T1-BE3, Q17 MMBF170, Q18 SI2337DS-T1-BE3, Q19 MMBF170, Q2 MMBF170, Q20 SI2337DS-T1-BE3, Q21 MMBF170, Q22 SI2337DS-T1-BE3, Q23 MMBF170, Q25 SI2337DS-T1-BE3, Q5 SI2337DS-T1-BE3, Q6 MMBF170, Q7 SI2337DS-T1-BE3, Q8 MMBF170, Q9 SI2337DS-T1-BE3

Commit message: Update schematic
Parts:
- removed AIR+_st1, GPIO2_Button, GPIO4_Button, R2D_Button1, TSON_Button: 7914J-1-000E, 7914J1000E, symbol 7914J-1-000E:7914J-1-000E
- removed AIR+_st2, GPIO2_Button, GPIO4_Button, R2D_Button2, TSON_Button: VFJD1105W-5C63A-TR, LEDC3216X195N, symbol VFJD1105W-5C63A-TR:VFJD1105W-5C63A-TR
- removed PS1: TEN_40-1211E, TEN401211E, symbol TEN_40-1211E:TEN_40-1211E
- removed R19, R28, R33, R59: 21.5k, EPSA_lib:RESC3216X70N, symbol EPSA_lib:Résistance RK73H2BLTDD2152F
- removed R21, R27, R32, R58: 15k, EPSA_lib:RESC3216X70N, symbol EPSA_lib:Résistance RK73H2BLTDD2152F
- removed V1: 5, symbol EPSA_lib:VSOURCE
- added C3: 4.7u, EPSA_lib:CAPC2012X130N, symbol EPSA_lib:Condensateur 0805Y1000104JXT
- added GREEN2, GREEN3, GREEN4, GREEN6, GREEN7: VFJD1105W-5C63A-TR, LEDC3216X195N, symbol VFJD1105W-5C63A-TR:VFJD1105W-5C63A-TR
- added IC3: TPS7B8633QDDARQ1, SOIC127P600X170-9N, symbol Régulateur de Tension Linéaire:TPS7B8633QDDARQ1
- added J6: 6P Droit 22-11-2062, EPSA_lib:HDRV6W87P0X254_1X6_1509X635X1092P, symbol EPSA_lib:6P Droit 22-11-2062
- added R39, R40, R41, R43, R44: 21.5k, EPSA_lib:RESC3216X70N, symbol EPSA_lib:Résistance RK73H2BLTDD2152F
- added R46, R47, R48, R50, R51: 11k, EPSA_lib:RESC3216X70N, symbol EPSA_lib:Résistance RK73H2BLTDD2152F
- added R73: 13.3k, EPSA_lib:RESC3216X70N, symbol EPSA_lib:Résistance RK73H2BLTDD2152F
- added R74: 2k, EPSA_lib:RESC3216X70N, symbol EPSA_lib:Résistance RK73H2BLTDD2152F
- added S11, S12, S7, S8, S9: 7914J-1-000E, 7914J1000E, symbol 7914J-1-000E:7914J-1-000E
- R10: renamed from R5; value 15k -> 11k
- R11: renamed from R7; value 15k -> 11k
- R12: renamed from R17; value 15k -> 11k
- R13: renamed from R14; value 15k -> 11k
- R45: renamed from R56; value 15k -> 11k
- R49: renamed from R23; value 15k -> 11k
- R56: renamed from R10; value 15k -> 11k
- R57: renamed from R46; value 15k -> 11k
- R58: renamed from R74; value 15k -> 11k
- R59: renamed from R76; value 15k -> 11k
- R60: value 15k -> 4.7k
- R61: value 21.5k -> 4.7k
- R8: renamed from R4; value 15k -> 11k
- R9: renamed from R1; value 15k -> 11k
- renumbered AIR+ to BLUE1, AIR- to BLUE2, BrakeLight to BLUE3, BuzzerR2D to BLUE4, Precharge to BLUE5, Decharge to BLUE6, GPIO1 to BLUE7, GPIO3 to BLUE8, C4 to C1, C3 to C2, AIR-_st2 to GREEN1, RRWSS to GREEN10, RRWSS to GREEN11, DryMode1 to GREEN5, FRWSS to GREEN8, FLWSS to GREEN9, Alimentation_12V to J1, SPI_SDCard to J10, J1 to J11, VCC_MCU to J2, Wheel_Speed_Sensors_Out to J3, Wheel_Speed_Sensors_In to J4, Analog_Out to J5, Digital_In to J7, Digital_Out to J8, CAN1 to J9, Q21 to Q1, Q22 to Q10, Q5 to Q11, Q25 to Q12, Q18 to Q13, Q16 to Q14, Q7 to Q15, Q9 to Q16, Q23 to Q2, Q15 to Q3, Q2 to Q4, Q19 to Q5, Q17 to Q6, Q6 to Q7, Q20 to Q9, R9 to R1, R63 to R14, R66 to R15, R48 to R16, R16 to R17, R54 to R18, R51 to R19, R3 to R2, R18 to R20, R29 to R21, R64 to R22, R67 to R23, R49 to R24, R11 to R25, R55 to R26, R52 to R27, R25 to R28, R30 to R29, R2 to R3, R65 to R30, R68 to R31, R50 to R32, R24 to R33, R62 to R34, R53 to R35, R26 to R36, R31 to R37, R57 to R38, R6 to R4, R22 to R42, R8 to R5, R70 to R52, R73 to R53, R75 to R54, R77 to R55, R20 to R6, R15 to R7, R44 to R72, 12V1 to RED1, S9 to S1, S1 to S10, FRWSS to S13, FLWSS to S14, RRWSS to S15, RLWSS to S16, S8 to S17, S2 to S18, S3 to S19, S10 to S2, S4 to S20, S12 to S3, S11 to S4, AIR-_st1 to S6
Connections:
- net 12V: now also S13.2 (-_2), S14.2 (-_2), S15.2 (-_2), S16.2 (-_2), S6.2 (-_2), IC3.7 (EN), IC3.8 (IN), S11.1 (-_1), S11.2 (-_2), S12.1 (-_1), S12.2 (-_2), S7.1 (-_1), S7.2 (-_2), S8.1 (-_1), S8.2 (-_2), S9.1 (-_1), S9.2 (-_2)
- net 5V: now also IC3.1 (OUT), R73.1
- net AIR+_st: now also R38.1, R45.2
- net AIR-_st: now also R39.1, R46.2; no longer R38.1, R45.2
- net CAN1H: now also R60.2
- net CAN1L: now also R61.1
- net FLWSS: no longer S18.2
- net FLWSS_in: now also S18.2
- net FLWSS_out: now also S18.3
- net FRWSS: no longer S17.2
- net FRWSS_in: now also S17.2
- net FRWSS_out: now also S17.3
- net GND: now also C3.1, IC3.5 (GND_1), IC3.9 (GND_2), R46.1, R47.1, R48.1, R50.1, R51.1, R74.2; no longer R60.1
- net GPIO2: now also R43.1, R50.2
- net GPIO4: now also R44.1, R51.2
- net R2D_Button: now also R41.1, R48.2; no longer R60.2, R61.1
- net RLWSS: no longer S20.2
- net RLWSS_in: now also S20.2
- net RLWSS_out: now also S20.3
- net RRWSS: no longer S19.2
- net RRWSS_in: now also S19.2
- net RRWSS_out: now also S19.3
- net TSON_Button: now also R40.1, R47.2
- net at R53.2: now also GREEN9.1 (K); no longer S14.3 (+_1)
- net at R52.2: now also GREEN8.1 (K); no longer S13.3 (+_1)
- net at S13.4 (+_2): now also GREEN8.2 (A), S13.3 (+_1); no longer GREEN8.1 (K)
- net RBPS_EXT: now reaches S4.3
- net RBPS_EXT: now also J6.4
- net at GREEN10.1 (K): now also R54.2; no longer S15.4 (+_2)
- net at GREEN10.2 (A): now also S15.3 (+_1), S15.4 (+_2); no longer S15.2 (-_2)
- net at GREEN11.1 (K): now also R55.2; no longer S16.4 (+_2)
- net at GREEN11.2 (A): now also S16.3 (+_1), S16.4 (+_2); no longer S16.2 (-_2)
- net at S14.4 (+_2): now also GREEN9.2 (A), S14.3 (+_1); no longer GREEN9.1 (K)
- net at R61.2: now also R60.1, C3.2
- net at GREEN1.1 (K): now also R38.2; no longer S6.4 (+_2)
- net at GREEN1.2 (A): now also S6.3 (+_1), S6.4 (+_2); no longer S6.2 (-_2)
- net APPS2_EXT: now reaches S2.3
- net APPS2_EXT: now also J6.3
- net ADC5_EXT: now reaches S5.3
- net ADC5_EXT: now also J6.6
- net APPS1_EXT: now reaches S1.3
- net APPS1_EXT: now also J6.2
- net FBPS_EXT: now reaches S3.3
- net FBPS_EXT: now also J6.1
- new net: GREEN4.1 (K), R41.2
- new net: GREEN4.2 (A), S9.3 (+_1), S9.4 (+_2)
- new net: GREEN2.1 (K), R39.2
- new net: IC3.2 (FB/NC), R73.2, R74.1
- new net: GREEN7.1 (K), R44.2
- new net: GREEN3.1 (K), R40.2
- new net: GREEN2.2 (A), S7.3 (+_1), S7.4 (+_2)
- new net: GREEN3.2 (A), S8.3 (+_1), S8.4 (+_2)
- new net: GREEN6.1 (K), R43.2
- new net: GREEN6.2 (A), S11.3 (+_1), S11.4 (+_2)
- new net: GREEN7.2 (A), S12.3 (+_1), S12.4 (+_2)
- no-connect marks 30 -> 34
Other:
- note added: "Sorties Analogiques"
- note added: "Sorties Compteurs"
- note removed: "Entrées Analogiques"
- note removed: "Entrées Compteurs"
- moved on the sheet: BLUE1, BLUE2, BLUE4, BLUE5, BLUE6, BLUE7, C1, GREEN1, GREEN10, GREEN11, GREEN5, GREEN8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

Commit message: Routage Support de programmation VCU
Parts:
- added C6: 2.2u, EPSA_lib:CAPC2012X130N, symbol EPSA_lib:Condensateur 0805Y1000104JXT
- added C7: 1u, EPSA_lib:CAPC2012X130N, symbol EPSA_lib:Condensateur 0805Y1000104JXT
- added J9: 2P Droit 2-11-2022, EPSA_lib:MOLEX_22-11-2022, symbol EPSA_lib:2P Droit 2-11-2022
- renumbered J9 to J10, J10 to J11, J11 to J12
Connections:
- net 12V: now also C6.2
- net 5V: now also C7.2
- net CAN1RX: now also J9.1
- net CAN1TX: now also J9.2
- net GND: now also C6.1, C7.1
Other:
- moved on the sheet: J10

Commit message: Routage Final
Parts:
- removed S1, S10, S17, S18, S19, S2, S20, S3, S4, S5: 100SP1T1B4M2QE, 100SP1T1B4M2QE, symbol 100SP1T1B4M2QE:100SP1T1B4M2QE
- removed S11, S12, S13, S14, S15, S16, S6, S7, S8, S9: 7914J-1-000E, 7914J1000E, symbol 7914J-1-000E:7914J-1-000E
- removed VR1, VR2, VR3, VR4, VR5: PTV09A-4015U-A503, PTV09A4015UA503, symbol Potentiomètre:PTV09A-4015U-A503
- added RV1, RV2, RV3, RV4, RV5: R_Potentiometer, PTV09A4015UA503, symbol Device:R_Potentiometer
- added SW1, SW10, SW17, SW18, SW19, SW2, SW20, SW3, SW4, SW5: 100SP1T1B4M2QE, 100SP1T1B4M2QE, symbol Switch:SW_Nidec_CAS-120A1
- added SW11, SW12, SW13, SW14, SW15, SW16, SW6, SW7, SW8, SW9: 7914J-1-000E, 7914J1000E, symbol Switch:SW_MEC_5E
Connections:
- net 12V: now also RV1.1, RV2.1, RV3.1, RV4.1, RV5.1, SW10.3 (A), SW11.1, SW11.2, SW12.1, SW12.2, SW13.1, SW13.2, SW14.1, SW14.2, SW15.1, SW15.2, SW16.1, SW16.2, SW6.1, SW6.2, SW7.1, SW7.2, SW8.1, SW8.2, SW9.1, SW9.2
- net ADC5: now also SW5.2 (B)
- net ADC5_EXT: now also SW5.3 (A)
- net APPS1: now also SW1.2 (B)
- net APPS1_EXT: now also SW1.3 (A)
- net APPS2: now also SW2.2 (B)
- net APPS2_EXT: now also SW2.3 (A)
- net FBPS: now also SW3.2 (B)
- net FBPS_EXT: now also SW3.3 (A)
- net FLWSS_in: now also SW18.2 (B)
- net FLWSS_out: now also SW18.3 (A)
- net FRWSS_in: now also SW17.2 (B)
- net FRWSS_out: now also SW17.3 (A)
- net GND: now also RV1.3, RV2.3, RV3.3, RV4.3, RV5.3, SW10.1 (C)
- net RBPS: now also SW4.2 (B)
- net RBPS_EXT: now also SW4.3 (A)
- net RLWSS_in: now also SW20.2 (B)
- net RLWSS_out: now also SW20.3 (A)
- net RRWSS_in: now also SW19.2 (B)
- net RRWSS_out: now also SW19.3 (A)
- net at R53.1, R57.2: now also SW18.1 (C)
- net at R52.1, R56.2: now also SW17.1 (C)
- net at R13.1, R7.1: now also SW5.1 (C)
- net at R7.2: now also RV5.2
- net at R2.2: now also RV1.2
- net at GREEN8.2 (A): now also SW13.3 (K), SW13.4 (A)
- net at R11.1, R5.1: now also SW4.1 (C)
- net at R55.1, R59.2: now also SW20.1 (C)
- net at GREEN10.2 (A): now also SW15.3 (K), SW15.4 (A)
- net at R3.1, R9.1: now also SW2.1 (C)
- net at R3.2: now also RV2.2
- net at R54.1, R58.2: now also SW19.1 (C)
- net at GREEN4.2 (A): now also SW9.3 (K), SW9.4 (A)
- net at GREEN11.2 (A): now also SW16.3 (K), SW16.4 (A)
- net at R10.1, R4.1: now also SW3.1 (C)
- net at GREEN9.2 (A): now also SW14.3 (K), SW14.4 (A)
- net at GREEN2.2 (A): now also SW7.3 (K), SW7.4 (A)
- net at GREEN3.2 (A): now also SW8.3 (K), SW8.4 (A)
- net at GREEN1.2 (A): now also SW6.3 (K), SW6.4 (A)
- net at R4.2: now also RV3.2
- net at GREEN6.2 (A): now also SW11.3 (K), SW11.4 (A)
- net at R2.1, R8.1: now also SW1.1 (C)
- net at R5.2: now also RV4.2
- net at GREEN7.2 (A): now also SW12.3 (K), SW12.4 (A)
- net at GREEN5.2 (A): now also SW10.2 (B)
- no-connect marks 34 -> 24

Commit message: Fin de stage
Parts:
- R1: value 21.5k -> 18k
- R2, R3, R39, R4, R40, R41, R42, R43, R44, R5, R52, R53, R54, R55, R6, R7: value 21.5k -> 22k
- R47: value 11k -> 22k
- R73: value 13.3k -> 15k
- R74: value 2k -> 2.2k
